File: sdr_sdri/ddr_soc.kicad_sch (KiCad schematic)
At the start: 0 parts

Commit message: add some connection to fpga ddr
Parts:
- added R? (x2): R_US, symbol Device:R_US
- added U?: Zynq-7010_7020, symbol Zynq7000:Zynq-7010_7020
Connections:
- new net DDR3_A0: U?.N2 (PS_DDR_A0_502)
- new net DDR3_A1: U?.K2 (PS_DDR_A1_502)
- new net DDR3_A10: U?.F5 (PS_DDR_A10_502)
- new net DDR3_A11: U?.G4 (PS_DDR_A11_502)
- new net DDR3_A12: U?.E4 (PS_DDR_A12_502)
- new net DDR3_A13: U?.D4 (PS_DDR_A13_502)
- new net DDR3_A14: U?.F4 (PS_DDR_A8_502)
- new net DDR3_A2: U?.M3 (PS_DDR_A2_502)
- new net DDR3_A3: U?.K3 (PS_DDR_A3_502)
- new net DDR3_A4: U?.M4 (PS_DDR_A4_502)
- new net DDR3_A5: U?.L1 (PS_DDR_A5_502)
- new net DDR3_A6: U?.L4 (PS_DDR_A6_502)
- new net DDR3_A7: U?.K4 (PS_DDR_A7_502)
- new net DDR3_A8: U?.F4 (PS_DDR_A8_502)
- new net DDR3_A9: U?.J4 (PS_DDR_A9_502)
- new net DDR3_D0: U?.C3 (PS_DDR_DQ0_502)
- new net DDR3_D1: U?.B3 (PS_DDR_DQ1_502)
- new net DDR3_D10: U?.G3 (PS_DDR_DQ10_502)
- new net DDR3_D11: U?.H3 (PS_DDR_DQ11_502)
- new net DDR3_D12: U?.J3 (PS_DDR_DQ12_502)
- new net DDR3_D13: U?.H2 (PS_DDR_DQ13_502)
- new net DDR3_D14: U?.H1 (PS_DDR_DQ14_502)
- new net DDR3_D15: U?.J1 (PS_DDR_DQ15_502)
- new net DDR3_D16: U?.P1 (PS_DDR_DQ16_502)
- new net DDR3_D17: U?.P3 (PS_DDR_DQ17_502)
- new net DDR3_D18: U?.R3 (PS_DDR_DQ18_502)
- new net DDR3_D19: U?.R1 (PS_DDR_DQ19_502)
- new net DDR3_D2: U?.A2 (PS_DDR_DQ2_502)
- new net DDR3_D20: U?.T4 (PS_DDR_DQ20_502)
- new net DDR3_D21: U?.U4 (PS_DDR_DQ21_502)
- new net DDR3_D22: U?.U2 (PS_DDR_DQ22_502)
- new net DDR3_D23: U?.U3 (PS_DDR_DQ23_502)
- new net DDR3_D24: U?.V1 (PS_DDR_DQ24_502)
- new net DDR3_D25: U?.Y3 (PS_DDR_DQ25_502)
- new net DDR3_D26: U?.W1 (PS_DDR_DQ26_502)
- new net DDR3_D27: U?.Y4 (PS_DDR_DQ27_502)
- new net DDR3_D28: U?.Y2 (PS_DDR_DQ28_502)
- new net DDR3_D29: U?.W3 (PS_DDR_DQ29_502)
- new net DDR3_D3: U?.A4 (PS_DDR_DQ3_502)
- new net DDR3_D30: U?.V2 (PS_DDR_DQ30_502)
- new net DDR3_D31: U?.V3 (PS_DDR_DQ31_502)
- new net DDR3_D4: U?.D3 (PS_DDR_DQ4_502)
- new net DDR3_D5: U?.D1 (PS_DDR_DQ5_502)
- new net DDR3_D6: U?.C1 (PS_DDR_DQ6_502)
- new net DDR3_D7: U?.E1 (PS_DDR_DQ7_502)
- new net DDR3_D8: U?.E2 (PS_DDR_DQ8_502)
- new net DDR3_D9: U?.E3 (PS_DDR_DQ9_502)
- new net DDR3_DM0: U?.A1 (PS_DDR_DM0_502)
- new net DDR3_DM1: U?.F1 (PS_DDR_DM1_502)
- new net DDR3_DM2: U?.T1 (PS_DDR_DM2_502)
- new net DDR3_DM3: U?.Y1 (PS_DDR_DM3_502)
- new net DDR3_DQS0_N: U?.C2 (PS_DDR_DQS_P0_502)
- new net DDR3_DQS0_P: U?.B2 (PS_DDR_DQS_N0_502)
- new net DDR3_DQS1_N: U?.G2 (PS_DDR_DQS_P1_502)
- new net DDR3_DQS1_P: U?.F2 (PS_DDR_DQS_N1_502)
- new net DDR3_DQS2_N: U?.R2 (PS_DDR_DQS_P2_502)
- new net DDR3_DQS2_P: U?.T2 (PS_DDR_DQS_N2_502)
- new net DDR3_DQS3_N: U?.W5 (PS_DDR_DQS_P3_502)
- new net DDR3_DQS3_P: U?.W4 (PS_DDR_DQS_N3_502)
- new net DDR_CKE: U?.N3 (PS_DDR_CKE_502)
- new net DDR_CKN: U?.M2 (PS_DDR_CKN_502)
- new net DDR_CLKP: U?.L2 (PS_DDR_CKP_502)
- new net DDR_ODT: U?.N5 (PS_DDR_ODT_502)
- new net DDR_VRN: R?.2, U?.H5 (PS_DDR_VRP_502)
- new net DDR_VRP: R?.2, U?.G5 (PS_DDR_VRN_502)
- new net GND: R?.1
