File: sdr_sdri/PowerSOC.kicad_sch (KiCad schematic)
At the start: 30 parts

Commit message: mer
Parts:
- added C? (x23): 470nF, symbol Device:C
- added C? (x13): 4.7uF, symbol Device:C
- added C? (x6): 100uF, symbol Device:C
- added C?: 10uF, symbol Device:C
- added J?: Conn_01x02_Male, symbol Connector:Conn_01x02_Male
- added L?: 600, symbol Device:L_Ferrite
- added R?: 0, symbol Device:R_US
- added U?: Zynq-7010_7020, symbol Zynq7000:Zynq-7010_7020
Connections:
- net GND: now also C?.2, C?.2, C?.2, C?.2, C?.2, C?.2, C?.2, C?.2, C?.2, C?.2, C?.2, C?.2, C?.2, C?.2, C?.2, C?.2, C?.2, C?.2, C?.2, C?.2, C?.2, C?.2, C?.2, C?.2, C?.2, C?.2, C?.2, C?.2, C?.2, C?.2, C?.2, C?.2, C?.2, C?.2, C?.2, C?.2, C?.2, C?.2, C?.2, C?.2, C?.2, C?.2, C?.2, J?.2 (Pin_2), U?.A18 (GND), U?.A8 (GND), U?.B1 (GND), U?.B11 (GND), U?.C14 (GND), U?.C4 (GND), U?.C9 (GND), U?.D17 (GND), U?.E10 (GND), U?.E20 (GND), U?.F3 (GND), U?.F7 (GND), U?.G10 (GND), U?.G12 (GND), U?.G16 (GND), U?.H11 (GND), U?.H13 (GND), U?.H19 (GND), U?.H7 (GND), U?.H9 (GND), U?.J12 (GND), U?.J2 (GND), U?.J8 (GND), U?.K11 (GND), U?.K13 (GND), U?.K15 (GND), U?.K5 (GND), U?.K7 (GND), U?.L12 (GND), U?.L18 (GND), U?.L8 (GND), U?.M1 (GND), U?.M11 (GND), U?.M13 (GND), U?.M7 (GND), U?.N10 (GND), U?.N12 (GND), U?.N14 (GND), U?.N4 (GND), U?.N8 (GND), U?.P11 (GND), U?.P13 (GND), U?.P17 (GND), U?.P7 (GND), U?.P9 (GND), U?.R12 (GND), U?.R20 (GND), U?.R8 (GND), U?.T13 (GND), U?.T3 (GND), U?.T7 (GND), U?.U16 (GND), U?.U6 (GND), U?.V19 (GND), U?.V9 (GND), U?.W12 (GND), U?.W2 (GND), U?.Y15 (GND), U?.Y5 (GND)
- net VCC1V0: now also U?.G11 (VCCBRAM), U?.G7 (VCCPINT), U?.H10 (VCCBRAM), U?.J7 (VCCPINT), U?.L7 (VCCPINT), U?.N7 (VCCPINT), U?.P8 (VCCPINT), U?.R7 (VCCPINT), C?.1, C?.1, C?.1, C?.1, C?.1, C?.1, C?.1, C?.1, C?.1, C?.1, C?.1, C?.1, C?.1
- net VCC1V8: now also U?.A13 (VCCO_MIO1_501), U?.B16 (VCCO_MIO1_501), U?.D12 (VCCO_MIO1_501), U?.E15 (VCCO_MIO1_501), U?.F8 (VCCPAUX), U?.G9 (VCCPAUX), U?.H8 (VCCPAUX), U?.K8 (VCCPAUX), U?.M8 (VCCPAUX), C?.1, C?.1, C?.1, C?.1, C?.1, C?.1, C?.1, C?.1, C?.1, C?.1, C?.1, C?.1, L?.2, R?.2
- net VCC3V3: now also U?.B6 (VCCO_MIO0_500), U?.D7 (VCCO_MIO0_500), C?.1, C?.1, C?.1, C?.1
- net VCC1V5: now reaches U?.A3 (VCCO_DDR_502)
- net VCC1V5: now also U?.D2 (VCCO_DDR_502), U?.E5 (VCCO_DDR_502), U?.G1 (VCCO_DDR_502), U?.H4 (VCCO_DDR_502), U?.L3 (VCCO_DDR_502), U?.P2 (VCCO_DDR_502), U?.R5 (VCCO_DDR_502), U?.U1 (VCCO_DDR_502), U?.V4 (VCCO_DDR_502), C?.1, C?.1, C?.1, C?.1, C?.1, C?.1, C?.1, C?.1, C?.1, C?.1, C?.1, C?.1
- net at U?.F11 (VCCBATT_0): now also J?.1 (Pin_1), R?.1
- net VCCPLL: now reaches U?.G8 (VCCPLL)
- net VCCPLL: now also C?.1, C?.1, L?.1
Other:
- moved on the sheet: C?, U?H
