File: sdr_sdri/Bank500.kicad_sch (KiCad schematic)
At the start: 4 parts

Commit message: menambahkan connecsi k
Parts:
- removed C?: 0.1uF, symbol Device:C
- removed R? (x2): 80, symbol Device:R_US
- removed U?: Zynq-7010_7020, symbol Zynq7000:Zynq-7010_7020
- added U? (x2): Zynq-7010_7020, symbol Zynq7000:Zynq-7010_7020
Connections:
- new net USB1HS_CLK: U?.A11 (PS_MIO36_501)
- new net USB1HS_D0: U?.A14 (PS_MIO32_501)
- new net USB1HS_D1: U?.D15 (PS_MIO33_501)
- new net USB1HS_D2: U?.A12 (PS_MIO34_501)
- new net USB1HS_D3: U?.F12 (PS_MIO35_501)
- new net USB1HS_D4: U?.C16 (PS_MIO28_501)
- new net USB1HS_D5: U?.A10 (PS_MIO37_501)
- new net USB1HS_D6: U?.E13 (PS_MIO38_501)
- new net USB1HS_D7: U?.C18 (PS_MIO39_501)
- new net USB1HS_DIR: U?.C13 (PS_MIO29_501), U?.D14 (PS_MIO40_501)
- new net USB1HS_NXT: U?.E12 (PS_MIO42_501), U?.E16 (PS_MIO31_501)
- new net USB1HS_STP: U?.C15 (PS_MIO30_501), U?.C17 (PS_MIO41_501)

Commit message: Add interface
Parts:
- added C?: 1uF, symbol Device:C
- added C?: 0.1uF, symbol Device:C
- added R? (x2): 1K, symbol Device:R_US
- added R?: 10K, symbol Device:R_US
Connections:
- net USB1HS_DIR: no longer U?.D14 (PS_MIO40_501)
- net USB1HS_NXT: no longer U?.E12 (PS_MIO42_501)
- net USB1HS_STP: no longer U?.C17 (PS_MIO41_501)
- net SDIO0_D2: now reaches U?.A9 (PS_MIO43_501)
- net PS_WARMRESET_INn: now reaches U?.B10 (PS_SRST_B_501)
- net SDIO0_WP: now reaches U?.B14 (PS_MIO47_501)
- net SDIO0_D4: now reaches U?.B15 (PS_MIO45_501)
- net SDIO0_CD: now reaches U?.D16 (PS_MIO46_501)
- net at U?.E11 (PS_MIO_VREF_501): now also C?.2, R?.1, R?.2
- net SDIO0_D3: now reaches U?.F13 (PS_MIO44_501)
- net at U?.C7 (PS_POR_B_500): now also C?.2, R?.2
- net PS_CLK: now reaches U?.E7 (PS_CLK_500)
- new net GNDD: C?.1, C?.1, R?.2
- new net SDIO0_CLK: U?.D14 (PS_MIO40_501)
- new net SDIO0_CMD: U?.C17 (PS_MIO41_501)
- new net SDIO0_D1: U?.E12 (PS_MIO42_501)
- new net VDDIO_500_PS: R?.1
- new net VDDIO_501_PS: R?.1
