File: sdr_sdri/interfes.kicad_sch (KiCad schematic)
At the start: 21 parts

Commit message: Add interface
Parts:
- added C?: 0.1uF, symbol Device:C
- added C?: 10uF, symbol Device:C
- added U?: W25Q128JVS, Package_SO:SOIC-8_5.23x5.23mm_P1.27mm, symbol Memory_Flash:W25Q128JVS
Connections:
- net GNDD: now also C?.2, C?.2, U?.4 (GND)
- new net +3.3V: C?.1, C?.1, U?.8 (VCC)
- new net QSP0I_CS0: U?.1 (~{CS})
- new net QSP0I_D0: U?.5 (DI(IO0))
- new net QSP0I_D1: U?.2 (DO(IO1))
- new net QSP0I_D2: U?.3 (IO2)
- new net QSP0I_D3: U?.7 (IO3)
- new net QSP0I_SCK: U?.6 (CLK)
